Commit message: [panthera] IK URDF: hand mass 0.6965 -> 1.10 kg per side for Dex5-1P
g1_body29_hand14.urdf describes the Dex3-1 hand: 0.6965 kg per side, of which
left/right_hand_palm_link carries 0.37283854 kg. A Dex5-1P is 1.1 kg. The IK's
gravity feed-forward (sol_tauff = pin.rnea with v = a = 0) is therefore about
20 % low on the shoulder-pitch and elbow joints, which is the difference between
holding a reach pose and sagging into it.

Raises only the two palm-link masses, by 0.40345 kg each, to 0.77629255. Inertia
tensors are deliberately left alone: we do not have a measured inertia for the
Dex5-1P, and a wrong tensor is worse than a slightly optimistic one for a link
this close to the wrist axis. CRLF line endings preserved (the file is CRLF).

Measured with tools/ik_smoke.py, 200 warm-started steps of the same slow oval
robot_arm_ik.__main__ walks, seeded so both runs follow an identical trajectory,
with g1_29_model_cache.pkl deleted in between (it pickles the inertias, so a stale
cache hides the edit entirely):

  full-model total mass    30.580234 -> 31.387142 kg   (+0.806908 = 2 x 0.40345)
  non-converged solves     0/200 before, 0/200 after
  solve time               mean 1.60 -> 1.53 ms, max 41.62 -> 19.12 ms
  max |q_post - q_base|    0.000000 rad -- identical pose, so the torque delta below
                           is purely the added mass

  tauff at the fixed reach pose (N*m):
    left_shoulder_pitch    -5.25620 -> -6.60533   (+1.34913)
    left_elbow             -3.23122 -> -4.30628   (+1.07507)
    right_shoulder_pitch   -5.08206 -> -6.39088   (+1.30883)
    right_elbow            -3.08893 -> -4.12405   (+1.03512)

File: assets/g1/g1_body29_hand14.urdf (robot description, URDF)
Before this commit: robot g1, 53 links, 52 joints
Links:
- link left_hand_palm_link: mass 0.37283854 -> 0.77629255
- link right_hand_palm_link: mass 0.37283854 -> 0.77629255

Commit message: [panthera] IK URDF: hand mass 1.10 -> 0.79 kg per side for the RH56E2
G5 set the palm mass for a Dex5-1P at 1.10 kg per side. That hand is not fitted. The
Inspire RH56E2-T1 weighs 790 g +/- 10 g, so the palm link goes 0.77629255 -> 0.46633854
and the per-side total 1.1000 -> 0.7900 kg. Two <mass> values, CRLF preserved, inertias
and every other link untouched.

Not reverted to stock. Upstream drives Inspire hands with the unmodified
g1_body29_hand14.urdf, whose 0.6965 kg per side models a Dex3, and 790 g is a measured
number from the vendor's own spec sheet -- close to the Dex3 but not equal to it. Using a
real number costs nothing and 0.0935 kg per side is not noise at the shoulder.

Source caveat: the 790 g figure is from the RH56E2 spec sheet, NOT from the RH56DFTP
manual, which gives gripping forces in grams but never states the hand's own mass. If
Inspire publishes a mass for the E2 specifically, prefer it.

Gravity feed-forward at the fixed reach pose, 0/200 non-converged in every run:

  joint          stock 0.6965   Dex5 1.10   RH56E2 0.79   vs stock
  L_sh_pitch          -5.2562     -6.6053       -5.5689     -0.3127
  L_elbow             -3.2312     -4.3063       -3.4804     -0.2491
  R_sh_pitch          -5.0821     -6.3909       -5.3854     -0.3033
  R_elbow             -3.0889     -4.1240       -3.3288     -0.2399
  |tauff| sum         28.1053     36.2018       29.9817

Every joint lands between the stock and Dex5 values, which is the expected ordering for a
mass between them. Model total 30.767 kg; palm parent-joint mass reads 0.55091501 kg per
side in Pinocchio (the palm link plus its fixed-joint children).

Worth noting for the overheating question: shoulder pitch carries the largest gravity
feed-forward of any arm joint, and the Dex5 assumption over-stated the extra load there
by about 4x (+1.35 N*m instead of +0.31). unitree_sdk2_python issue #129 reports G1
shoulder-pitch overheating with an Inspire FTP hand on arm_sdk.

The Dex5 lane stays parked, not deleted: robot_hand_unitree.py, the Dex5 assets, the
hand_config dex5 model and all four Dex5 tests remain and still pass under HAND_MODEL=dex5.
--ee dex5 still parses. PR #321 is verified work and remains useful if a Dex5 ever
arrives; deleting a verified path to make room for a new one loses the verification.

File: assets/g1/g1_body29_hand14.urdf (robot description, URDF)
Before this commit: robot g1, 53 links, 52 joints
Links:
- link left_hand_palm_link: mass 0.77629255 -> 0.46633854
- link right_hand_palm_link: mass 0.77629255 -> 0.46633854
